File: afe_230v_16a/afe_230v_16a.kicad_pcb (KiCad board)
At the start: 2 copper layers, 67.7 x 86.4 mm, 0 parts

Commit message: 011425 end of day
Parts:
- added REF**: BlackPill, STM-32:YAAJ_BlackPill_SWD_1, F.Cu at (217.6, 73.5)
Other:
- board text added: "keepout areas for BC 71,6 OT-U11"
