File: afe_230v_16a/afe_230v_16a.kicad_sch (KiCad schematic)
At the start: 71 parts, among them J4 MCV 1,5/ 6-G-3,81, P1 06-14-03_rectifier, U1 ${SIM.PARAMS}, U17 1_element_2_current, U2 AD8538, U20 watt_hour_meter_bidirectional, U21 3w_ne, U3 AD8538, U4 AQH3223A, U5 ACS711xLCTR-25AB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

Commit message: 011425 end of day
Parts:
- added U9: YAAJ_BlackPill, STM-32:YAAJ_BlackPill_SWD_2, symbol YAAJ_BlackPill:YAAJ_BlackPill
Connections:
- net 3V3: now also U9.16 (3V3)
- net Earth: now also U9.17 (GND), U9.18 (GND)
- net at U20.: now also T16.
- net at T16.: now also T17.; no longer U20.
- net at C8.: now also T10.
- net at T10.: now also T8.; no longer C8.
- net at C7.: now also C3., P1., T8., U8.
- net at T17.: now also C12.; no longer T16.
- net at T7.: now also C3.
- net at T11.: now also C9.; no longer T9.
- net at C9.: no longer T11.
- net at U21.: no longer C12.
- new net: T11., T9.
- new net: C12., U21.
- now unconnected: P1., U8.
