File: bc_71,6_edgecuts/bc_71,6_edgecuts.kicad_pcb (KiCad board)
At the start: 2 copper layers, 668 x 168.4 mm, 14 parts, among them J1 MKDSN 2,5/ 6-5,08, J2 MKDS 1,5/ 6, J5 HBUS16, J6 pinheader_2x6_socket, J9 Conn_01x04_STlink_pinheader

Commit message: adjusted inter-pcb-connector location, added edgecuts pcb2,3,4,8,9
Parts:
- removed the J6 at (-135.9, 151.8)
- moved J6 2.97 mm to (213.8, 87.8)
- moved J6 2.97 mm to (115.2, 108.1)
Routing:
- net (no net): track 114.3 -> 437.0 mm
Other:
- outline, holes or cut-outs redrawn
- board text added: "pcb4 BC 71,6 UT11 13.6mm clearance from pcb1"
- board text added: "pcb8 BC 71,6 27,6 clearance"
- board text added: "pcb9 BC 71,6 30,45 clearance"
- board text removed: "BC 71,6 UT11 pcb4 13.6mm clearance"
- board text removed: "bc71,6 UT11 pcb8"
- board text removed: "bc71,6 pcb9"
