File: afe_230v_16a_main/afe_230v_16a.kicad_sch (KiCad schematic)
At the start: 85 parts, among them J1 MKDSN 2,5/ 6-5,08, J2 MKDS 1,5/ 6, J5 HBUS16, J6 pinheader_2x6_socket, J9 Conn_01x04_STlink_pinheader, P1 06-14-03_rectifier, U1 ${SIM.PARAMS}, U10 BlackPill_F4_SWI, U17 1_element_2_current, U2 AD8538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

Commit message: changed r20 net
Connections:
- net at R22.1, R24.1, U1.1: now also R19.2, R20.1; no longer R19.1
- net at U20.: now also T16.
- net at T16.: now also T17.; no longer U20.
- net at R20.2, R23.1, R25.1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: now also R21.2; no longer R21.1
- net at U2.4 (-): now also R21.1; no longer R21.2
- net at C8.: now also T10.
- net at T10.: now also T8.; no longer C8.
- net at C7.: now also C3., P1., T8., U8.
- net at T17.: now also C12.; no longer T16.
- net at T7.: now also C3.
- net at T11.: now also C9.; no longer T9.
- net at C9.: no longer T11.
- net at U21.: no longer C12.
- new net: R19.1, U1.4 (-)
- new net: T11., T9.
- new net: C12., U21.
- now unconnected: P1., U8.
Other:
- moved on the sheet: R19, R20, R21
