File: afe_230v_16a_main/afe_230v_16a.kicad_sch (KiCad schematic)
At the start: 85 parts, among them J1 MKDSN 2,5/ 6-5,08, J2 MKDS 1,5/ 6, J5 HBUS16, J6 pinheader_2x6_socket, J9 Conn_01x04_STlink_pinheader, P1 06-14-03_rectifier, U1 ${SIM.PARAMS}, U10 BlackPill_F4_SWI, U17 1_element_2_current, U2 AD8538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

Commit message: added JLC BOM & CPL
Parts:
- C1, C10, C2, C4, C5, C6: footprint Capacitor_SMD:C_0603_1608Metric_Pad1.08x0.95mm_HandSolder -> Capacitor_SMD:C_0402_1005Metric
Connections:
- net at U20.: now also T16.
- net at T16.: now also T17.; no longer U20.
- net at C8.: now also T10.
- net at T10.: now also T8.; no longer C8.
- net at C7.: now also C3., P1., T8., U8.
- net at T17.: now also C12.; no longer T16.
- net at T7.: now also C3.
- net at T11.: now also C9.; no longer T9.
- net at C9.: no longer T11.
- net at U21.: no longer C12.
- new net: T11., T9.
- new net: C12., U21.
- now unconnected: P1., U8.
Changed lines of the file:
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@@
 			)
 		)
-		(property "Footprint" "Capacitor_SMD:C_0603_1608Metric_Pad1.08x0.95mm_HandSolder"
+		(property "Footprint" "Capacitor_SMD:C_0402_1005Metric"
 			(at 342.5952 125.73 0)
 			(effects
@@
 			)
 		)
-		(property "Footprint" "Capacitor_SMD:C_0603_1608Metric_Pad1.08x0.95mm_HandSolder"
+		(property "Footprint" "Capacitor_SMD:C_0402_1005Metric"
 			(at 331.1652 125.73 0)
 			(effects
@@
 			)
 		)
-		(property "Footprint" "Capacitor_SMD:C_0603_1608Metric_Pad1.08x0.95mm_HandSolder"
+		(property "Footprint" "Capacitor_SMD:C_0402_1005Metric"
 			(at 308.3052 125.73 0)
 			(effects
@@
 			)
 		)
-		(property "Footprint" "Capacitor_SMD:C_0603_1608Metric_Pad1.08x0.95mm_HandSolder"
+		(property "Footprint" "Capacitor_SMD:C_0402_1005Metric"
 			(at 319.7352 125.73 0)
 			(effects
@@
 			)
 		)
-		(property "Footprint" "Capacitor_SMD:C_0603_1608Metric_Pad1.08x0.95mm_HandSolder"
+		(property "Footprint" "Capacitor_SMD:C_0402_1005Metric"
 			(at 148.2852 91.44 0)
 			(effects
@@
 			)
 		)
-		(property "Footprint" "Capacitor_SMD:C_0603_1608Metric_Pad1.08x0.95mm_HandSolder"
+		(property "Footprint" "Capacitor_SMD:C_0402_1005Metric"
 			(at 148.2852 49.53 0)
 			(effects

Commit message: updated buildnote
Connections:
- net at U20.: now also T16.
- net at T16.: now also T17.; no longer U20.
- net at C8.: now also T10.
- net at T10.: now also T8.; no longer C8.
- net at C7.: now also C3., P1., T8., U8.
- net at T17.: now also C12.; no longer T16.
- net at T7.: now also C3.
- net at T11.: now also C9.; no longer T9.
- net at C9.: no longer T11.
- net at U21.: no longer C12.
- new net: T11., T9.
- new net: C12., U21.
- now unconnected: P1., U8.
Other:
- note added: "R29: shunt resistor"
- note added: "R39 connects dgnd to gnd"
Changed lines of the file:
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@@
+		)
+	)
+	(text "R39 connects dgnd to gnd"
+		(exclude_from_sim no)
+		(at 373.634 120.142 0)
+		(effects
+			(font
+				(size 1.27 1.27)
+			)
 		)
 	)
@@
 		(effects
 			(font
+				(size 1.27 1.27)
+			)
+		)
+	)
+	(text "R29: shunt resistor"
+		(exclude_from_sim no)
+		(at 126.746 198.374 90)
+		(effects
+			(font

Commit message: upgraded to kicad 9.0.6
Connections:
- net at U20.: now also T16.
- net at T16.: now also T17.; no longer U20.
- net at C8.: now also T10.
- net at T10.: now also T8.; no longer C8.
- net at C7.: now also C3., P1., T8., U8.
- net at T17.: now also C12.; no longer T16.
- net at T7.: now also C3.
- net at T11.: now also C9.; no longer T9.
- net at C9.: no longer T11.
- net at U21.: no longer C12.
- new net: T11., T9.
- new net: C12., U21.
- now unconnected: P1., U8.
Changed lines of the file:
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@@
 (kicad_sch
-	(version 20231120)
+	(version 20250114)
 	(generator "eeschema")
-	(generator_version "8.0")
+	(generator_version "9.0")
 	(paper "B")
+	(rectangle
+		(start 278.13 146.05)
+		(end 351.79 176.53)
+		(stroke
+			(width 0)
+			(type default)
+		)
+		(fill
+			(type none)
+		)
+	)
+	(rectangle
+		(start 288.29 170.18)
+		(end 297.18 175.26)
+		(stroke
+			(width 0)
+			(type default)
+		)
+		(fill
+			(type none)
+		)
+	)
+	(rectangle
+		(start 260.35 137.16)
+		(end 396.24 228.6)
+		(stroke
+			(width 0)
+			(type default)
+		)
+		(fill
+			(type none)
+		)
+	)
+	(text "Note: AMC1200 may allow high side"
+		(exclude_from_sim no)
+		(at 160.274 221.742 0)
+		(effects
+			(font
+				(size 1.27 1.27)
+			)
+		)
+	)
+	(text "AC Grid\nConnection"
+		(exclude_from_sim no)
+		(at 388.366 219.456 0)
+		(effects
+			(font
+				(size 1.27 1.27)
+			)
+		)
+	)
+	(text "Block Diagram"
+		(exclude_from_sim no)
+		(at 384.81 142.24 0)
+		(effects
+			(font
+				(size 1.27 1.27)
+			)
+		)
+	)
+	(text "Low side current sense\n(Prefer High side and need a part for higher common mode rejection)"
+		(exclude_from_sim no)
+		(at 177.546 217.678 0)
+		(effects
+			(font
+				(size 1.27 1.27)
+			)
+		)
+	)
+	(text "R39 connects dgnd to gnd"
+		(exclude_from_sim no)
+		(at 373.634 120.142 0)
+		(effects
+			(font
+				(size 1.27 1.27)
+			)
+		)
+	)
+	(text "KO"
+		(exclude_from_sim no)
+		(at 310.642 166.878 0)
+		(effects
+			(font
+				(size 1.27 1.27)
+			)
+		)
+	)
+	(text "(1) Vsense\n(1) Isense\n(1) K0"
+		(exclude_from_sim no)
+		(at 341.376 151.13 0)
+		(effects
+			(font
+				(size 1.27 1.27)
+			)
+		)
+	)
+	(text "Current measurement"
+		(exclude_from_sim no)
+		(at 293.116 168.402 0)
+		(effects
+			(font
+				(size 1.27 1.27)
+			)
+		)
+	)
+	(text "Energy\nMeter"
+		(exclude_from_sim no)
+		(at 355.854 218.44 0)
+		(effects
+			(font
+				(size 1.27 1.27)
+			)
+		)
+	)
+	(text "LOAD"
+		(exclude_from_sim no)
+		(at 322.58 207.01 0)
+		(effects
+			(font
+				(size 1.27 1.27)
+			)
+		)
+	)
+	(text "Thermomagnetic\nCircuit\nBreaker"
+		(exclude_from_sim no)
+		(at 370.586 219.964 0)
+		(effects
+			(font
+				(size 1.27 1.27)
+			)
+		)
+	)
+	(text "LOAD"
+		(exclude_from_sim no)
+		(at 279.4 200.66 0)
+		(effects
+			(font
+				(size 1.27 1.27)
+			)
+		)
+	)
+	(text "R29: shunt resistor"
+		(exclude_from_sim no)
+		(at 126.746 198.374 90)
+		(effects
+			(font
+				(size 1.27 1.27)
+			)
+		)
+	)
+	(text "Contactor/\nRelay"
+		(exclude_from_sim no)
+		(at 303.276 208.28 0)
+		(effects
+			(font
+				(size 1.27 1.27)
+			)
+		)
+	)
 	(junction
 		(at 325.12 187.96)
@@
 		)
 	)
-	(rectangle
-		(start 278.13 146.05)
-		(end 351.79 176.53)
-		(stroke
-			(width 0)
-			(type default)
-		)
-		(fill
-			(type none)
-		)
-	)
-	(rectangle
-		(start 288.29 170.18)
-		(end 297.18 175.26)
-		(stroke
-			(width 0)
-			(type default)
-		)
-		(fill
-			(type none)
-		)
-	)
-	(rectangle
-		(start 260.35 137.16)
-		(end 396.24 228.6)
-		(stroke
-			(width 0)
-			(type default)
-		)
-		(fill
-			(type none)
-		)
-	)
-	(text "Note: AMC1200 may allow high side"
-		(exclude_from_sim no)
-		(at 160.274 221.742 0)
-		(effects
-			(font
-				(size 1.27 1.27)
-			)
-		)
-	)
-	(text "AC Grid\nConnection"
-		(exclude_from_sim no)
-		(at 388.366 219.456 0)
-		(effects
-			(font
-				(size 1.27 1.27)
-			)
-		)
-	)
-	(text "Block Diagram"
-		(exclude_from_sim no)
-		(at 384.81 142.24 0)
-		(effects
-			(font
-				(size 1.27 1.27)
-			)
-		)
-	)
-	(text "Low side current sense\n(Prefer High side and need a part for higher common mode rejection)"
-		(exclude_from_sim no)
-		(at 177.546 217.678 0)
-		(effects
-			(font
-				(size 1.27 1.27)
-			)
-		)
-	)
-	(text "R39 connects dgnd to gnd"
-		(exclude_from_sim no)
-		(at 373.634 120.142 0)
-		(effects
-			(font
-				(size 1.27 1.27)
-			)
-		)
-	)
-	(text "KO"
-		(exclude_from_sim no)
-		(at 310.642 166.878 0)
-		(effects
-			(font
-				(size 1.27 1.27)
-			)
-		)
-	)
-	(text "(1) Vsense\n(1) Isense\n(1) K0"
-		(exclude_from_sim no)
-		(at 341.376 151.13 0)
-		(effects
-			(font
-				(size 1.27 1.27)
-			)
-		)
-	)
-	(text "Current measurement"
-		(exclude_from_sim no)
-		(at 293.116 168.402 0)
-		(effects
-			(font
-				(size 1.27 1.27)
-			)
-		)
-	)
-	(text "Energy\nMeter"
-		(exclude_from_sim no)
-		(at 355.854 218.44 0)
-		(effects
-			(font
-				(size 1.27 1.27)
-			)
-		)
-	)
-	(text "LOAD"
-		(exclude_from_sim no)
-		(at 322.58 207.01 0)
-		(effects
-			(font
-				(size 1.27 1.27)
-			)
-		)
-	)
-	(text "Thermomagnetic\nCircuit\nBreaker"
-		(exclude_from_sim no)
-		(at 370.586 219.964 0)
-		(effects
-			(font
-				(size 1.27 1.27)
-			)
-		)
-	)
-	(text "LOAD"
-		(exclude_from_sim no)
-		(at 279.4 200.66 0)
-		(effects
-			(font
-				(size 1.27 1.27)
-			)
-		)
-	)
-	(text "R29: shunt resistor"
-		(exclude_from_sim no)
-		(at 126.746 198.374 90)
-		(effects
-			(font
-				(size 1.27 1.27)
-			)
-		)
-	)
-	(text "Contactor/\nRelay"
-		(exclude_from_sim no)
-		(at 303.276 208.28 0)
-		(effects
-			(font
-				(size 1.27 1.27)
-			)
-		)
-	)
 	(label "A1"
 		(at 383.54 34.29 0)
@@
 		)
 	)
+	(embedded_fonts no)
 )
